File: LogicBoard 3GE/LogicBoard 3GE.kicad_sch (KiCad schematic)
At the start: 156 parts, among them IC201 2363, IC204 2114, IC205 2114, IC206 68A09, IC207 6522, IC208 AY3-8912, IC301 MC1408, IC302 CD4052B, IC303 LF347, IC304 LF353, IC305 4066, J201 CART, J202 DB9_Male, J203 DB9_Male, J204 Power, J301 Video, J302 Audio, Q301 2N3906, Q302 2N3906, Q303 2N3904, SW201 Reset, U202 74LS00, U203 74LS32, Y201 6MHz

Commit message: Add files via upload
Parts:
- renumbered U202 to IC202, U203 to IC203
Other:
- moved on the sheet: IC202A, IC202B, IC202C, IC202D, IC203B, IC203C, IC203D, R226

Commit message: Add files via upload
Parts:
- removed C330: 1nF, Capacitor_THT:C_Disc_D5.0mm_W2.5mm_P5.00mm, symbol Device:C_Small
- added R306, R308, R310, R312: 680, Vectrex LogicBoard:R_Axial_DIN0207_L6.3mm_D2.5mm_P12.70mm_Horizontal, symbol Device:R_Small
- added R329: 6.8k, Vectrex LogicBoard:R_Axial_DIN0207_L6.3mm_D2.5mm_P12.70mm_Horizontal, symbol Device:R_Small
- added R330: 3.3k, Vectrex LogicBoard:R_Axial_DIN0207_L6.3mm_D2.5mm_P12.70mm_Horizontal, symbol Device:R_Small
- added R336: 1M, Vectrex LogicBoard:R_Axial_DIN0207_L6.3mm_D2.5mm_P12.70mm_Horizontal, symbol Device:R_Small
- C201, C204, C205, C206, C207, C208, C209, C223, C301, C302, C314, C316, C317, C320, C321, C324, C326, C327, C328: Mouser 581-SR215C104K -> 581-SR215C104k
- C210, C222: Mouser 581-SR215A220KARTR1 -> 581-SR215A220kARTR1
- C323: Mouser 647-UKT1E4R7MDD1TD -> 647-UkT1E4R7MDD1TD
- R201: value 22K -> 22k
- R202, R203, R206, R207, R209, R210, R322, R324: value 3.3K -> 3.3k; Mouser 603-CFR-25JR-523K3 -> 603-CFR-25JR-523k3
- R204, R205: value 3.3K -> 3.3k
- R301, R304, R305: value 2.7K 1% -> 2.7k 1%; Mouser 603-MFR-25FRF522K49 -> 603-MFR-25FRF522k49
- R302: value 10K -> 10k; Mouser 531-PT10H-5K-S -> 531-PT10H-5k-S
- R303: value 3.6K 1% -> 3.6k 1%; Mouser 603-MFR-25FRF52-2K61 -> 603-MFR-25FRF52-2k61
- R307, R309, R311, R313: value 330K -> 330k; Mouser 603-CFR-25JR-52-330K -> 603-CFR-25JR-52-330k
- R314, R315: value 2.2K -> 2.2k; Mouser 603-CFR-25JR-522K2 -> 603-CFR-25JR-522k2
- R316, R319: value 10K 1% -> 10k 1%; Mouser 603-MFR-25FRF5210K -> 603-MFR-25FRF5210k
- R323, R325: value 15K -> 15k; Mouser 603-CFR-25JR-5215K -> 603-CFR-25JR-5215k
- R326, R333, R335: value 10K -> 10k; Mouser 531-PT10H-10K-S -> 531-PT10H-10k-S
- R327, R344, R345, R346: value 33K -> 33k; Mouser 603-CFR-25JR-52-33K -> 603-CFR-25JR-52-33k
- R338, R339: value 4.7K -> 4.7k; Mouser 603-CFR-25JR-524K7 -> 603-CFR-25JR-524k7
- R340: value 10K -> 10k; Mouser 603-CFR-25JR-5210K -> 603-CFR-25JR-5210k
- R341, R342, R343: value 1K -> 1k; Mouser 603-CFR-25JR-521K -> 603-CFR-25JR-521k
- SW201: footprint Inductor_THT:L_Axial_L7.0mm_D3.3mm_P12.70mm_Horizontal_Fastron_MICC -> TestPoint:TestPoint_Bridge_Pitch5.08mm_Drill1.3mm
Connections:
- net +5VA is gone; now on net +5V: C202.1, C212.1, C234.1, C236.2, C301.2, C314.2, C320.2, FB202.2, IC301.13 (VCC), IC302.16 (VDD), IC303.4 (V+), IC304.8 (V+), IC305.14 (VDD), J202.7, J203.7, J204.2 (Pin_2), R301.2, R304.2, R333.1, R335.1
- net +5V: now also R336.1
- net GNDA: now also R330.2
- net POT0: now also R312.2; no longer C232.2, J203.5
- net POT1: now also R310.2; no longer C233.2, J203.6
- net POT2: now also R308.1; no longer C230.1, J202.5
- net POT3: now also R306.1, R336.2; no longer C231.1, J202.6
- net at R327.2: now also R329.1, R330.1; no longer IC302.11 (X3)
- net A0R: no longer names the net of IC206.8 (A0), R214.2
- net A1R: no longer names the net of IC206.9 (A1), R215.2
- net Q: no longer names the net of IC206.35 (Q)
- new net: C230.1, J202.5, R308.2
- new net: C232.2, J203.5, R312.1
- new net: C233.2, J203.6, R310.1
- new net: IC302.11 (X3), R329.2
- new net: C231.1, J202.6, R306.2
- no-connect marks 4 -> 5
Other:
- note added: "+5V ANALOGIC"
- note added: "-5V ANALOGIC"
- note added: "ANALOGIC GROUND"
- note removed: "+5V ANALOGIQUE"
- note removed: "-5V ANALOGIQUE"
- note removed: "ANALOGIQUE GROUND"
- note removed: "TO IC301 PIN3 ONLY"
- moved on the sheet: C214, C215, C216, C217, C218, C219, C220, C221, C224, C228, C229, C230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

Commit message: FIRQ & CA1
Replace Label SW3 & SW7 by FIRQ & CA1 for more visibility.
Connections:
- net SW3 renamed FIRQ
- net SW7 renamed CA1
Other:
- moved on the sheet: C205, IC205
