File: CRTBoard/CRTBoard.kicad_sch (KiCad schematic)
At the start: 17 parts

Commit message: correction to the LM379 on the PowerBoard
- Convert to Kicad 8
- Correction to the LM379 on the PowerBoard and C405,C406,R404,R411
- Correct value of F101
Other:
- moved on the sheet: CRT
